File: Weight Scale/Hardware/WEIGHT_PCB/AD7190.kicad_sch (KiCad schematic)
At the start: 1 part, among them IC1 AD7190BRUZ

Commit message: update schematics
Parts:
- added C1, C14, C2, C4, C5: 100nF, Capacitor_SMD:C_0402_1005Metric_Pad0.74x0.62mm_HandSolder, symbol Device:C
- added C10, C9: 1uF, Capacitor_SMD:C_0603_1608Metric, symbol Device:C
- added C11, C12, C7, C8: 10nF, Capacitor_SMD:C_0603_1608Metric, symbol Device:C
- added C13: 10uF, Capacitor_SMD:C_0402_1005Metric_Pad0.74x0.62mm_HandSolder, symbol Device:C
- added C3, C6: 10uF, Capacitor_SMD:C_0805_2012Metric, symbol Device:C
- added D1, D3: CDSOD323-T05, PCM_Diode_SMD_AKL:D_SOD-323, symbol PCM_Diode_TVS_AKL:CDSOD323-T05
- added D2, D4, D5, D6, D7: CG0603MLC-12LE, BM_KiCad_Library:VARC1608X55N, symbol BM_KiCad_library:CG0603MLC-12LE
- added FB1, FB2: MPZ1608S331ATA00, Inductor_SMD:L_0603_1608Metric, symbol Device:FerriteBead
- added FL1, FL2, FL3, FL4, FL5, FL6: NFE31PT101C1E9L, BM_KiCad_Library:NFE31, symbol BM_KiCad_library:NFE31PT101C1E9L
- added FL10, FL11, FL7, FL8, FL9: NFM18CC101R1C3D, BM_KiCad_Library:FIL_NFM18CC101R1C3D, symbol BM_KiCad_library:NFM18CC101R1C3D
- added R1: 2.2 Ω, PCM_Resistor_SMD_AKL:R_0402_1005Metric_Pad0.72x0.64mm, symbol Device:R
- added R10, R6: 10, PCM_Resistor_SMD_AKL:R_0402_1005Metric, symbol Device:R
- added R11, R2: 0, PCM_Resistor_SMD_AKL:R_0402_1005Metric, symbol Device:R
- added R3, R4, R5, R7, R8, R9: 100, PCM_Resistor_SMD_AKL:R_0402_1005Metric, symbol Device:R
Connections:
- net GNDA: now reaches IC1.10 (AINCOM)
- net GNDA: now also IC1.18 (AGND), C1.2, C11.1, C12.2, C13.2, C14.2, C2.2, C3.2, C4.2, C5.2, C6.2, C7.2, C8.2, D1.2 (A), D2.1, D3.2 (A), D4.1, D5.1, D6.1, D7.1, FL1.2 (GND_1), FL1.4 (GND_2), FL1.5 (GND_3), FL10.2, FL10.2_1, FL10.2_2, FL10.2_3, FL10.2_4, FL11.2, FL11.2_1, FL11.2_2, FL11.2_3, FL11.2_4, FL2.1 (IN), FL2.2 (GND_1), FL2.4 (GND_2), FL2.5 (GND_3), FL3.2 (GND_1), FL3.4 (GND_2), FL3.5 (GND_3), FL4.2 (GND_1), FL4.4 (GND_2), FL4.5 (GND_3), FL5.2 (GND_1), FL5.4 (GND_2), FL5.5 (GND_3), FL6.2 (GND_1), FL6.4 (GND_2), FL6.5 (GND_3), FL7.2, FL7.2_1, FL7.2_2, FL7.2_3, FL7.2_4, FL8.2, FL8.2_1, FL8.2_2, FL8.2_3, FL8.2_4, FL9.2, FL9.2_1, FL9.2_2, FL9.2_3, FL9.2_4
- net AIN1: now reaches IC1.11 (AIN1)
- net AIN1: now also C7.1, C9.1, R4.2
- net AIN2: now reaches IC1.12 (AIN2)
- net AIN2: now also C11.2, C9.2, R8.2
- net REFIN1-: now reaches IC1.15 (REFIN1(+))
- net REFIN1-: now also C10.2, C12.1, R10.2
- net REFIN1+: now reaches IC1.16 (REFIN1(-))
- net REFIN1+: now also C10.1, C8.1, R6.2
- net GND: now reaches IC1.19 (DGND)
- net AVDD: now reaches IC1.20 (AVDD)
- net AVDD: now also C2.1, C3.1, C4.1, C5.1, C6.1, FB1.2, FL1.1 (IN)
- net +3.3V: now reaches IC1.21 (DVDD)
- net +3.3V: now also C13.1, C14.1
- net at IC1.22 (~{SYNC}): now also FL11.1
- net at IC1.23 (DOUT/~{RDY}): now also FL9.1
- net at IC1.24 (DIN): now also FL7.1
- net at IC1.3 (SCLK): now also FL8.3
- net at IC1.4 (~{CS}): now also FL10.3
- new net: D6.2, FL3.1 (IN), R3.2
- new net: FB1.1, R1.2
- new net: D1.1 (K), D2.2, FB2.1, FL1.3 (OUT)
- new net: D7.2, FL5.1 (IN), R7.2
- new net: FL5.3 (OUT), R8.1
- new net: D5.2, FL6.1 (IN), R9.2
- new net: FL6.3 (OUT), R10.1
- new net: D4.2, FL4.1 (IN), R5.2
- new net: FL4.3 (OUT), R6.1
- new net: FL3.3 (OUT), R4.1
- new net !CS: FL10.1
- new net !SYNC: FL11.3
- new net +5V_A: C1.1, R1.1
- new net MISO: FL9.3
- new net MOSI: FL7.3
- new net SCK: FL8.1
- new net SENSE+: R2.1, R5.1
- new net SENSE-: R11.2, R9.1
- new net SIGNAL+: R3.1
- new net SIGNAL-: R7.1
- new net VCEL+: FB2.2, R2.2
- new net VCEL-: D3.1 (K), FL2.3 (OUT), R11.1
- no-connect marks 0 -> 9
Other:
- note added: "FILTER"
- note added: "Note: Supply is VCEL"
- moved on the sheet: IC1

Commit message: update schematics
Changed lines of the file:
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@@
 			(font
 				(size 1.27 1.27)
+				(bold yes)
 			)
 			(justify left bottom)
@@
 				(size 1.27 1.27)
 				(thickness 0.1588)
+				(bold yes)
 			)
 			(justify right bottom)
@@
 				(size 1.27 1.27)
 				(thickness 0.1588)
+				(bold yes)
 			)
 			(justify right bottom)
@@
 				(size 1.27 1.27)
 				(thickness 0.1588)
+				(bold yes)
 			)
 			(justify left bottom)
@@
 				(size 1.27 1.27)
 				(thickness 0.1588)
+				(bold yes)
 			)
 			(justify left bottom)
@@
 				(size 1.27 1.27)
 				(thickness 0.1588)
+				(bold yes)
 			)
 			(justify left bottom)
@@
 			(font
 				(size 1.27 1.27)
+				(bold yes)
 			)
 			(justify right bottom)
@@
 				(size 1.27 1.27)
 				(thickness 0.1588)
+				(bold yes)
 			)
 			(justify right bottom)
@@
 				(size 1.27 1.27)
 				(thickness 0.1588)
+				(bold yes)
 			)
 			(justify right bottom)
@@
 				(size 1.27 1.27)
 				(thickness 0.1588)
+				(bold yes)
 			)
 			(justify right bottom)
@@
 			(font
 				(size 1.27 1.27)
+				(bold yes)
 			)
 			(justify left bottom)
@@
 				(size 1.27 1.27)
 				(thickness 0.1588)
+				(bold yes)
 			)
 			(justify left bottom)
@@
 				(size 1.27 1.27)
 				(thickness 0.1588)
+				(bold yes)
 			)
 			(justify left bottom)
@@
 			(font
 				(size 1.27 1.27)
+				(bold yes)
 			)
 			(justify left bottom)
@@
 				(size 1.27 1.27)
 				(thickness 0.1588)
+				(bold yes)
 			)
 			(justify left bottom)
@@
 				(size 1.27 1.27)
 				(thickness 0.1588)
+				(bold yes)
 			)
 			(justify left bottom)
@@
 				(size 1.27 1.27)
 				(thickness 0.1588)
+				(bold yes)
 			)
 			(justify left bottom)
@@
 				(size 1.27 1.27)
 				(thickness 0.1588)
+				(bold yes)
 			)
 			(justify right bottom)
@@
 				(size 1.27 1.27)
 				(thickness 0.1588)
+				(bold yes)
 			)
 			(justify right bottom)
@@
 				(size 1.27 1.27)
 				(thickness 0.1588)
+				(bold yes)
 			)
 			(justify right bottom)
@@
 				(size 1.27 1.27)
 				(thickness 0.1588)
+				(bold yes)
 			)
 			(justify right bottom)
@@
 			(font
 				(size 1.27 1.27)
+				(bold yes)
 			)
 			(justify right bottom)
@@
 				(size 1.27 1.27)
 				(thickness 0.1588)
-			)
-			(justify left bottom)
+				(bold yes)
+			)
+			(justify left bottom)

Commit message: update schematics
Other:
- note added: "Notes: Using Internal Clock of 4.92 MHz (+-4%) Using AIN1 and AIN2 as differential input channel"
Changed lines of the file:
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@@
+		)
+	)
+	(text "Notes:\nUsing Internal Clock of 4.92 MHz (+-4%)\nUsing AIN1 and AIN2 as differential input channel"
+		(exclude_from_sim no)
+		(at 84.074 188.976 0)
+		(effects
+			(font
+				(size 1.27 1.27)
+				(thickness 0.254)
+				(bold yes)
+			)
+			(justify left)
 		)
 	)
@@
 			(font
 				(size 1.27 1.27)
-				(bold yes)
+				(thickness 0.1588)
 			)
 			(justify left bottom)
@@
 				(size 1.27 1.27)
 				(thickness 0.1588)
-				(bold yes)
 			)
 			(justify right bottom)
@@
 				(size 1.27 1.27)
 				(thickness 0.1588)
-				(bold yes)
 			)
 			(justify right bottom)
@@
 				(size 1.27 1.27)
 				(thickness 0.1588)
-				(bold yes)
 			)
 			(justify left bottom)
@@
 				(size 1.27 1.27)
 				(thickness 0.1588)
-				(bold yes)
 			)
 			(justify left bottom)
@@
 				(size 1.27 1.27)
 				(thickness 0.1588)
-				(bold yes)
 			)
 			(justify left bottom)
@@
 			(font
 				(size 1.27 1.27)
-				(bold yes)
+				(thickness 0.1588)
 			)
 			(justify right bottom)
@@
 				(size 1.27 1.27)
 				(thickness 0.1588)
-				(bold yes)
 			)
 			(justify right bottom)
@@
 				(size 1.27 1.27)
 				(thickness 0.1588)
-				(bold yes)
 			)
 			(justify right bottom)
@@
 				(size 1.27 1.27)
 				(thickness 0.1588)
-				(bold yes)
 			)
 			(justify right bottom)
@@
 			(font
 				(size 1.27 1.27)
-				(bold yes)
+				(thickness 0.1588)
 			)
 			(justify left bottom)
@@
 				(size 1.27 1.27)
 				(thickness 0.1588)
-				(bold yes)
 			)
 			(justify left bottom)
@@
 				(size 1.27 1.27)
 				(thickness 0.1588)
-				(bold yes)
 			)
 			(justify left bottom)
@@
 			(font
 				(size 1.27 1.27)
-				(bold yes)
+				(thickness 0.1588)
 			)
 			(justify left bottom)
@@
 				(size 1.27 1.27)
 				(thickness 0.1588)
-				(bold yes)
 			)
 			(justify left bottom)
@@
 				(size 1.27 1.27)
 				(thickness 0.1588)
-				(bold yes)
 			)
 			(justify left bottom)
@@
 				(size 1.27 1.27)
 				(thickness 0.1588)
-				(bold yes)
 			)
 			(justify left bottom)
@@
 				(size 1.27 1.27)
 				(thickness 0.1588)
-				(bold yes)
 			)
 			(justify right bottom)
@@
 				(size 1.27 1.27)
 				(thickness 0.1588)
-				(bold yes)
 			)
 			(justify right bottom)
@@
 				(size 1.27 1.27)
 				(thickness 0.1588)
-				(bold yes)
 			)
 			(justify right bottom)
@@
 				(size 1.27 1.27)
 				(thickness 0.1588)
-				(bold yes)
 			)
 			(justify right bottom)
@@
 			(font
 				(size 1.27 1.27)
-				(bold yes)
+				(thickness 0.1588)
 			)
 			(justify right bottom)
@@
 				(size 1.27 1.27)
 				(thickness 0.1588)
-				(bold yes)
 			)
 			(justify left bottom)
@@
 	)
 	(hierarchical_label "VCEL+"
-		(shape input)
+		(shape output)
 		(at 25.4 20.32 180)
 		(fields_autoplaced yes)
@@
 	)
 	(hierarchical_label "VCEL-"
-		(shape input)
+		(shape output)
 		(at 25.4 22.86 180)
 		(fields_autoplaced yes)
