File: Weight Scale/Hardware/WEIGHT_PCB/EEPROM.kicad_sch (KiCad schematic)
At the start: 1 part, among them IC3 AT24C04C-SSHM-T

Commit message: update schematics
Changed lines of the file:
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@@
+	(wire
+		(pts
+			(xy 30.48 30.48) (xy 40.64 30.48)
+		)
+		(stroke
+			(width 0)
+			(type default)
+		)
+	)
+	(wire
+		(pts
+			(xy 30.48 27.94) (xy 40.64 27.94)
+		)
+		(stroke
+			(width 0)
+			(type default)
+		)
+	)
 	(wire
 		(pts
@@
 		)
 	)
+	(label "SCL"
+		(at 40.64 27.94 0)
+		(fields_autoplaced yes)
+		(effects
+			(font
+				(size 1.27 1.27)
+			)
+			(justify left bottom)
+		)
+	)
 	(label "SDA"
 		(at 163.83 99.06 0)
@@
 			)
 			(justify left bottom)
+		)
+	)
+	(label "SDA"
+		(at 40.64 30.48 0)
+		(fields_autoplaced yes)
+		(effects
+			(font
+				(size 1.27 1.27)
+			)
+			(justify left bottom)
+		)
+	)
+	(hierarchical_label "SCL"
+		(shape bidirectional)
+		(at 30.48 27.94 180)
+		(fields_autoplaced yes)
+		(effects
+			(font
+				(size 1.27 1.27)
+			)
+			(justify right)
+		)
+	)
+	(hierarchical_label "SDA"
+		(shape bidirectional)
+		(at 30.48 30.48 180)
+		(fields_autoplaced yes)
+		(effects
+			(font
+				(size 1.27 1.27)
+			)
+			(justify right)
 		)
 	)
@@
 		(on_board yes)
 		(dnp no)
-		(property "Reference" "#PWR016"
+		(property "Reference" "#PWR043"
 			(at 170.18 105.41 0)
 			(effects
@@
 			(project "WEIGHT_PCB"
 				(path "/5fd124d5-f631-461d-96a1-dd77850b026f/8eeca3c0-ba26-48f9-96e8-6d33db4880af"
-					(reference "#PWR016")
+					(reference "#PWR043")
 					(unit 1)
 				)
@@
 		(on_board yes)
 		(dnp no)
-		(property "Reference" "#PWR014"
+		(property "Reference" "#PWR042"
 			(at 135.89 105.41 0)
 			(effects
@@
 			(project ""
 				(path "/5fd124d5-f631-461d-96a1-dd77850b026f/8eeca3c0-ba26-48f9-96e8-6d33db4880af"
-					(reference "#PWR014")
+					(reference "#PWR042")
 					(unit 1)
 				)
@@
 		(dnp no)
 		(fields_autoplaced yes)
-		(property "Reference" "#PWR015"
+		(property "Reference" "#PWR041"
 			(at 163.83 93.98 0)
 			(effects
@@
 			(project ""
 				(path "/5fd124d5-f631-461d-96a1-dd77850b026f/8eeca3c0-ba26-48f9-96e8-6d33db4880af"
-					(reference "#PWR015")
+					(reference "#PWR041")
 					(unit 1)
 				)

Commit message: update schematics
Changed lines of the file:
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@@
 			(font
 				(size 1.27 1.27)
+				(bold yes)
 			)
 			(justify left bottom)
@@
 			(font
 				(size 1.27 1.27)
+				(bold yes)
 			)
 			(justify left bottom)
@@
 			(font
 				(size 1.27 1.27)
+				(bold yes)
 			)
 			(justify left bottom)
@@
 			(font
 				(size 1.27 1.27)
+				(bold yes)
 			)
 			(justify left bottom)

Commit message: update schematics
Changed lines of the file:
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@@
 			(font
 				(size 1.27 1.27)
-				(bold yes)
+				(thickness 0.1588)
 			)
 			(justify left bottom)
@@
 			(font
 				(size 1.27 1.27)
-				(bold yes)
+				(thickness 0.1588)
 			)
 			(justify left bottom)
@@
 			(font
 				(size 1.27 1.27)
-				(bold yes)
+				(thickness 0.1588)
 			)
 			(justify left bottom)
@@
 			(font
 				(size 1.27 1.27)
-				(bold yes)
+				(thickness 0.1588)
 			)
 			(justify left bottom)
