File: Weight Scale/Hardware/WEIGHT_PCB/FT230XS.kicad_sch (KiCad schematic)
At the start: 7 parts, among them U1 FT230XS

Commit message: update schematics
Parts:
- added C39, C40: 10nF, Capacitor_SMD:C_0402_1005Metric, symbol Device:C
- added FB4: MPZ1608S331ATA00, Inductor_SMD:L_0603_1608Metric, symbol Device:FerriteBead
- added R24, R25: 10K, PCM_Resistor_SMD_AKL:R_0402_1005Metric_Pad0.72x0.64mm, symbol Device:R
- renumbered C4 to C22, C5 to C23, C6 to C24, C7 to C25, R6 to R20, R7 to R21
Connections:
- net GND: now also C39.2, C40.2, R25.1
- net at U1.11 (~{RESET}): now also C39.1, R24.1, R25.2
- new net: C40.1, FB4.2, R24.2
- new net VUSB: FB4.1
Other:
- note added: "RESET IS INVERTED"
- moved on the sheet: C24, C25, R20, R21

Commit message: update schematics
Parts:
- added D10, D11: LED, LED_SMD:LED_0603_1608Metric, symbol Device:LED
- added R26, R27: 270, PCM_Resistor_SMD_AKL:R_0402_1005Metric_Pad0.72x0.64mm, symbol Device:R
Connections:
- net +3.3V: now also U1.10 (3V3OUT), D10.2 (A), D11.2 (A)
- net RXD2: now reaches U1.1 (TXD)
- net RX_LED: now reaches U1.14 (CBUS1)
- net RX_LED: now also R26.1
- net TXD2: now reaches U1.4 (RXD)
- net TX_LED: now reaches U1.7 (CBUS2)
- net TX_LED: now also R27.1
- new net: D10.1 (K), R26.2
- new net: D11.1 (K), R27.2
- no-connect marks 0 -> 1
Other:
- note removed: "RESET IS INVERTED"
- moved on the sheet: C22, C23, FB4

Commit message: update schematics
Parts:
- added C24, C25: 100nF, Capacitor_SMD:C_0402_1005Metric_Pad0.74x0.62mm_HandSolder, symbol Device:C
- added IC4: SN74LVC1G08DCKRG4, BM_KiCad_Library:SC70-5, symbol BM_KiCad_library:SN74LVC1G08DCKRG4
- added RN1: EXB-38V103JV, BM_KiCad_Library:EXB38V472JV, symbol BM_KiCad_library:EXB-38V103JV
- D10: value LED -> RX_LED
- D11: value LED -> TX_LED
- renumbered C24 to C26, C25 to C27, C40 to C28, C39 to C29, R26 to R22, R27 to R23
Connections:
- net +3.3V: now also C24.1, C25.2, IC4.5 (VCC), RN1.5, RN1.6, RN1.7, RN1.8
- net GND: now also C24.2, C25.1, IC4.3 (GND)
- net RXD2: now also IC4.4 (Y); no longer U1.1 (TXD)
- net TXD2: now also RN1.2
- net at U1.2 (~{RTS}): now also RN1.3
- net at U1.6 (~{CTS}): now also RN1.4
- net RX_LED: no longer names the net of R22.1, U1.14 (CBUS1)
- net TX_LED: no longer names the net of R23.1, U1.7 (CBUS2)
- new net: IC4.1 (A), RN1.1, U1.1 (TXD)
- new net RXD_TTL: IC4.2 (B)
- no-connect marks 1 -> 2
Other:
- moved on the sheet: C22, C23, C26, C29, D10, D11
