File: Weight Scale/Hardware/WEIGHT_PCB/LIS2DH12TR.kicad_sch (KiCad schematic)
At the start: 3 parts, among them U2 LIS2DH12TR

Commit message: update schematics
Parts:
- renumbered C8 to C26, C9 to C27
Changed lines of the file:
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@@
 	)
 	(hierarchical_label "SCL"
-		(shape input)
+		(shape bidirectional)
 		(at 30.48 45.72 180)
 		(fields_autoplaced yes)
@@
 	)
 	(hierarchical_label "SDA"
-		(shape input)
+		(shape bidirectional)
 		(at 30.48 48.26 180)
 		(fields_autoplaced yes)
@@
 	)
 	(hierarchical_label "INT1_ACEL"
-		(shape input)
+		(shape output)
 		(at 30.48 50.8 180)
 		(fields_autoplaced yes)
@@
 		(dnp no)
 		(fields_autoplaced yes)
-		(property "Reference" "#PWR024"
+		(property "Reference" "#PWR049"
 			(at 120.65 90.17 0)
 			(effects
@@
 			(project "WEIGHT_PCB"
 				(path "/5fd124d5-f631-461d-96a1-dd77850b026f/45873352-bc65-475d-9863-8a0332d84f81"
-					(reference "#PWR024")
+					(reference "#PWR049")
 					(unit 1)
 				)
@@
 		(dnp no)
 		(fields_autoplaced yes)
-		(property "Reference" "#PWR022"
+		(property "Reference" "#PWR050"
 			(at 184.15 96.52 0)
 			(effects
@@
 			(project "WEIGHT_PCB"
 				(path "/5fd124d5-f631-461d-96a1-dd77850b026f/45873352-bc65-475d-9863-8a0332d84f81"
-					(reference "#PWR022")
+					(reference "#PWR050")
 					(unit 1)
 				)
@@
 		(dnp no)
 		(fields_autoplaced yes)
-		(property "Reference" "C8"
+		(property "Reference" "C26"
 			(at 181.61 83.82 0)
 			(effects
@@
 			(project "WEIGHT_PCB"
 				(path "/5fd124d5-f631-461d-96a1-dd77850b026f/45873352-bc65-475d-9863-8a0332d84f81"
-					(reference "C8")
+					(reference "C26")
 					(unit 1)
 				)
@@
 		(dnp no)
 		(fields_autoplaced yes)
-		(property "Reference" "C9"
+		(property "Reference" "C27"
 			(at 193.04 83.82 0)
 			(effects
@@
 			(project "WEIGHT_PCB"
 				(path "/5fd124d5-f631-461d-96a1-dd77850b026f/45873352-bc65-475d-9863-8a0332d84f81"
-					(reference "C9")
+					(reference "C27")
 					(unit 1)
 				)
@@
 		(dnp no)
 		(fields_autoplaced yes)
-		(property "Reference" "#PWR023"
+		(property "Reference" "#PWR051"
 			(at 163.83 113.03 0)
 			(effects
@@
 			(project ""
 				(path "/5fd124d5-f631-461d-96a1-dd77850b026f/45873352-bc65-475d-9863-8a0332d84f81"
-					(reference "#PWR023")
+					(reference "#PWR051")
 					(unit 1)
 				)
@@
 		(dnp no)
 		(fields_autoplaced yes)
-		(property "Reference" "#PWR021"
+		(property "Reference" "#PWR048"
 			(at 189.23 81.28 0)
 			(effects
@@
 			(project "WEIGHT_PCB"
 				(path "/5fd124d5-f631-461d-96a1-dd77850b026f/45873352-bc65-475d-9863-8a0332d84f81"
-					(reference "#PWR021")
+					(reference "#PWR048")
 					(unit 1)
 				)

Commit message: update schematics
Changed lines of the file:
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@@
 			(font
 				(size 1.27 1.27)
+				(bold yes)
 			)
 			(justify right bottom)
@@
 			(font
 				(size 1.27 1.27)
+				(bold yes)
 			)
 			(justify right bottom)
@@
 			(font
 				(size 1.27 1.27)
+				(bold yes)
 			)
 			(justify left bottom)
@@
 			(font
 				(size 1.27 1.27)
+				(bold yes)
 			)
 			(justify left bottom)
@@
 			(font
 				(size 1.27 1.27)
+				(bold yes)
 			)
 			(justify left bottom)
@@
 			(font
 				(size 1.27 1.27)
+				(bold yes)
 			)
 			(justify left bottom)

Commit message: update schematics
Parts:
- renumbered C26 to C30, C27 to C31
Changed lines of the file:
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@@
 			(font
 				(size 1.27 1.27)
-				(bold yes)
+				(thickness 0.1588)
 			)
 			(justify right bottom)
@@
 			(font
 				(size 1.27 1.27)
-				(bold yes)
+				(thickness 0.1588)
 			)
 			(justify right bottom)
@@
 			(font
 				(size 1.27 1.27)
-				(bold yes)
+				(thickness 0.1588)
 			)
 			(justify left bottom)
@@
 		(dnp no)
 		(fields_autoplaced yes)
-		(property "Reference" "#PWR049"
+		(property "Reference" "#PWR056"
 			(at 120.65 90.17 0)
 			(effects
@@
 			(project "WEIGHT_PCB"
 				(path "/5fd124d5-f631-461d-96a1-dd77850b026f/45873352-bc65-475d-9863-8a0332d84f81"
-					(reference "#PWR049")
+					(reference "#PWR056")
 					(unit 1)
 				)
@@
 		(dnp no)
 		(fields_autoplaced yes)
-		(property "Reference" "#PWR050"
+		(property "Reference" "#PWR057"
 			(at 184.15 96.52 0)
 			(effects
@@
 			(project "WEIGHT_PCB"
 				(path "/5fd124d5-f631-461d-96a1-dd77850b026f/45873352-bc65-475d-9863-8a0332d84f81"
-					(reference "#PWR050")
+					(reference "#PWR057")
 					(unit 1)
 				)
@@
 		(dnp no)
 		(fields_autoplaced yes)
-		(property "Reference" "C26"
+		(property "Reference" "C30"
 			(at 181.61 83.82 0)
 			(effects
@@
 			(project "WEIGHT_PCB"
 				(path "/5fd124d5-f631-461d-96a1-dd77850b026f/45873352-bc65-475d-9863-8a0332d84f81"
-					(reference "C26")
+					(reference "C30")
 					(unit 1)
 				)
@@
 		(dnp no)
 		(fields_autoplaced yes)
-		(property "Reference" "C27"
+		(property "Reference" "C31"
 			(at 193.04 83.82 0)
 			(effects
@@
 			(project "WEIGHT_PCB"
 				(path "/5fd124d5-f631-461d-96a1-dd77850b026f/45873352-bc65-475d-9863-8a0332d84f81"
-					(reference "C27")
+					(reference "C31")
 					(unit 1)
 				)
@@
 		(dnp no)
 		(fields_autoplaced yes)
-		(property "Reference" "#PWR051"
+		(property "Reference" "#PWR058"
 			(at 163.83 113.03 0)
 			(effects
@@
 			(project ""
 				(path "/5fd124d5-f631-461d-96a1-dd77850b026f/45873352-bc65-475d-9863-8a0332d84f81"
-					(reference "#PWR051")
+					(reference "#PWR058")
 					(unit 1)
 				)
@@
 		(dnp no)
 		(fields_autoplaced yes)
-		(property "Reference" "#PWR048"
+		(property "Reference" "#PWR055"
 			(at 189.23 81.28 0)
 			(effects
@@
 			(project "WEIGHT_PCB"
 				(path "/5fd124d5-f631-461d-96a1-dd77850b026f/45873352-bc65-475d-9863-8a0332d84f81"
-					(reference "#PWR048")
+					(reference "#PWR055")
 					(unit 1)
 				)
