File: Weight Scale/Hardware/WEIGHT_PCB/Voltage_Regulators.kicad_sch (KiCad schematic)
At the start: 17 parts, among them IC4 TPS7A2033PDBVR, IC5 TPS7A2050PDBVR, IC6 AOZ1280CI

Commit message: update schematics
Parts:
- renumbered IC6 to IC5, IC5 to IC6
Other:
- title: (none) -> Voltage Regulators
Changed lines of the file:
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@@
 	(paper "A4")
 	(title_block
+		(title "Voltage Regulators")
 		(date "2024-11-12")
 		(rev "0.01")
@@
 			(font
 				(size 1.27 1.27)
+				(bold yes)
 			)
 			(justify left bottom)
@@
 			(font
 				(size 1.27 1.27)
+				(bold yes)
 			)
 			(justify left bottom)
@@
 			(font
 				(size 1.27 1.27)
+				(bold yes)
 			)
 			(justify right bottom)
@@
 		(dnp no)
 		(fields_autoplaced yes)
-		(property "Reference" "IC5"
+		(property "Reference" "IC6"
 			(at 223.52 109.22 0)
 			(effects
@@
 		(dnp no)
 		(fields_autoplaced yes)
-		(property "Reference" "#PWR040"
+		(property "Reference" "#PWR057"
 			(at 218.44 135.89 0)
 			(effects
@@
 		(dnp no)
 		(fields_autoplaced yes)
-		(property "Reference" "IC6"
+		(property "Reference" "IC5"
 			(at 90.17 72.39 0)
 			(effects
@@
 		(dnp no)
 		(fields_autoplaced yes)
-		(property "Reference" "#PWR038"
+		(property "Reference" "#PWR053"
 			(at 256.54 90.17 0)
 			(effects

Commit message: update schematics
Parts:
- added D12: 1N5819, Diode_SMD:D_SOD-123, symbol PCM_Diode_Schottky_AKL:1N5819
- renumbered C28 to C32, C29 to C33, C30 to C34, C31 to C35, C32 to C36, C33 to C37, C34 to C38, C35 to C39, C36 to C40, C37 to C41, C38 to C42, IC4 to IC5, IC5 to IC6, IC6 to IC7, R22 to R26, R23 to R27
Connections:
- net GND: now also D12.2 (A)
- net at C34.2, IC6.6 (LX), L1.1: now also D12.1 (K)
