File: Weight Scale/Hardware/WEIGHT_PCB/microcontroller.kicad_sch (KiCad schematic)
At the start: 15 parts, among them IC2 STM32F303CCT7

Commit message: update schematics
Parts:
- added C21: 100nF, Capacitor_SMD:C_0402_1005Metric_Pad0.74x0.62mm_HandSolder, symbol Device:C
- added D9: LED, LED_SMD:LED_1206_3216Metric, symbol Device:LED
- added J1: FTSH-105-01-L-DV, BM_KiCad_Library:FTSH-105-XX-YYY-DV, symbol BM_KiCad_library:FTSH-105-01-L-DV
- added R13: 1K, PCM_Resistor_SMD_AKL:R_0402_1005Metric_Pad0.72x0.64mm_HandSolder, symbol Device:R
- added R17: 10K, PCM_Resistor_SMD_AKL:R_0402_1005Metric_Pad0.72x0.64mm_HandSolder, symbol Device:R
- added R18: 0, PCM_Resistor_SMD_AKL:R_0402_1005Metric_Pad0.72x0.64mm, symbol Device:R
- renumbered C11 to C15, C10 to C16, C12 to C17, C3 to C18, C1 to C19, C2 to C20, D1 to D8, FB1 to FB3, R1 to R12, R2 to R14, R4 to R15, R5 to R16, R3 to R19
Connections:
- net !KEY: now also IC2.31 (PA10); no longer IC2.32 (PA11)
- net +3.3V: now also J1.1, R13.1, R17.1
- net GND: now also C21.2, D9.1 (K), J1.3, J1.5
- net NRST: now also C21.1, R17.2, R18.2
- net SWDCLK: now also J1.4
- net SWDIO: now also J1.2
- net USB_DP: now reaches IC2.33 (PA12)
- net SYNC renamed !SYNC
- new net: D9.2 (A), R13.2
- new net: J1.10, R18.1
- new net USB_DN: IC2.32 (PA11)
Other:
- note added: "JTAG"
- moved on the sheet: C15, C16, C17, C18, C19, C20, D8, FB3, R12, R14, R15, R16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

Commit message: update schematics
Parts:
- D8, D9: footprint LED_SMD:LED_1206_3216Metric -> LED_SMD:LED_0603_1608Metric
Connections:
- net VBAT: no longer names the net of C18.1, IC2.1 (VBAT)
Other:
- note added: "3V3 LED FEEDBACK"
- note added: "CONFIGURABLE LED"
- note added: "DECOUPLING CAPACITORS"
- note added: "I2C PULL UP RESISTORS"
- note added: "JTAG CONNECTOR"
- note added: "PUSH BUTTON"
- note removed: "JTAG"
- moved on the sheet: D8, D9, FB3, R12, R13, R14, R15, R16, S1

Commit message: update schematics
Parts:
- renumbered R17 to R15, R15 to R16, R16 to R17
